File: Hardware/power-divider/power_divider.kicad_pcb (KiCad board)
At the start: 4 copper layers, 40 x 51.9 mm, 22 parts, among them J1 Conn_Coaxial, J2 Conn_Coaxial, J3 Conn_Coaxial

Commit message: Vias galore
Routing:
- net GND: track 0.08 -> 0.00 mm, vias 0 -> 151
Other:
- outline, holes or cut-outs redrawn

Commit message: Hans's gargantuine PR review has been fulfilled except for rebasing, removed unwanted sch file and README.md
Other:
- board text added: "1.6 mm FR4 Dk = 4.6 Green Soldermask No Silkscreen HASL Lead Free Order with Stencil"
Changed lines of the file:
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@@
     (effects (font (size 1 1) (thickness 0.15)))
+  )
+  (gr_text "1.6 mm FR4\nDk = 4.6\nGreen Soldermask\nNo Silkscreen\nHASL Lead Free\nOrder with Stencil" (at 156.337 55.753) (layer "F.Fab")
+    (effects (font (size 0.7 0.7) (thickness 0.1)) (justify left))
   )
   (via (at 135.992859 65.997532) (size 0.8) (drill 0.4) (layers "F.Cu" "B.Cu") (free) (net 1))
